File: lora_sensor_tag/power.kicad_sch (KiCad schematic)
At the start: 54 parts, among them J3 Li-ion_bat_conn, Q1 NPN, U5 TPS63070RNMR, U6 MCP73871-2CAI_ML, U8 MAX17048G_T10

Commit message: Comment and capasitor formfactor.
Parts:
- C40: footprint Capacitor_SMD:C_0603_1608Metric -> Capacitor_SMD:C_0402_1005Metric
Changed lines of the file:
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@@
 		)
 	)
+	(text_box "PG & FB connection order ???"
+		(exclude_from_sim no)
+		(at 224.79 21.59 0)
+		(size 8.89 10.16)
+		(margins 0.9525 0.9525 0.9525 0.9525)
+		(stroke
+			(width 0)
+			(type dot)
+		)
+		(fill
+			(type none)
+		)
+		(effects
+			(font
+				(size 0.762 0.762)
+			)
+			(justify left top)
+		)
+	)
 	(junction
 		(at 227.33 27.94)
@@
 			)
 		)
-		(property "Footprint" "Capacitor_SMD:C_0603_1608Metric"
+		(property "Footprint" "Capacitor_SMD:C_0402_1005Metric"
 			(at 220.6752 57.15 0)
 			(hide yes)
